Commit message: first test

File: urdf/camera.xacro (robot description, xacro)
@@ -1,10 +1,10 @@
 <?xml version="1.0"?>
-<robot xmlns:xacro="http://www.ros.org/wiki/xacro" name="my_robot">
-<xacro:macro name="head">
-    <link name="head_link">
+<robot xmlns:xacro="http://www.ros.org/wiki/xacro" name="growbot">
+<xacro:macro name="camera">
+    <link name="camera_link">
         <visual>
             <origin rpy="0 0 0" xyz="0 0 0"/>
             <geometry>
-                <mesh filename="package://tutorial/urdf/head.dae" scale="5 5 5"/>
+                <mesh filename="package://tutorial/urdf/camera.dae" scale="5 5 5"/>
             </geometry>
         </visual>
@@ -21,17 +21,17 @@
         </inertial>
     </link>
-    <joint name="base_to_head" type="continuous">
+    <joint name="base_to_camera" type="continuous">
         <axis xyz="0 0 1"/>  <!-- changes axis of rotation -->
         <parent link="base_link"/>
-        <child link="head_link"/>
+        <child link="camera_link"/>
         <origin rpy="0 0 0" xyz="0 0 .5"/> <!-- moves the child_frame with respect to parent_frame -->
         <limit effort="30" velocity="1.0"/>
     </joint>
-    <transmission name="head_transmission">
+    <transmission name="camera_transmission">
         <type>transmission_interface/SimpleTransmission</type>
-        <actuator name="$head_motor">
+        <actuator name="$camera_motor">
             <mechanicalReduction>1</mechanicalReduction>
         </actuator>
-        <joint name="base_to_head">
+        <joint name="base_to_camera">
             <hardwareInterface>hardware_interface/PositionJointInterface</hardwareInterface>
         </joint>

File: urdf/main.xacro (robot description, xacro)
@@ -1,6 +1,6 @@
 <?xml version="1.0"?>
-<robot xmlns:xacro="http://www.ros.org/wiki/xacro" name="my_robot">
-    <xacro:include filename="$(find tutorial)/urdf/arm.xacro" />
-    <xacro:include filename="$(find tutorial)/urdf/head.xacro" />
+<robot xmlns:xacro="http://www.ros.org/wiki/xacro" name="growbot">
+    <xacro:include filename="$(find tutorial)/urdf/wheel.xacro" />
+    <xacro:include filename="$(find tutorial)/urdf/camera.xacro" />
     <link name="base_link">
         <visual>
@@ -19,7 +19,7 @@
         </inertial>
     </link>
-    <xacro:arm prefix="right" length=".7" radius=".2" reflect="1" />
-    <xacro:arm prefix="left" length=".7" radius=".2" reflect="-1" />
-    <xacro:head />
+    <xacro:wheel prefix="right" length=".7" radius=".2" reflect="1" />
+    <xacro:wheel prefix="left" length=".7" radius=".2" reflect="-1" />
+    <xacro:camera />
     <!-- Add ROS plugin so we can interact with our robot -->
     <gazebo>

File: urdf/wheel.xacro (robot description, xacro)
@@ -1,8 +1,8 @@
 <?xml version="1.0"?>
-<robot xmlns:xacro="http://www.ros.org/wiki/xacro" name="my_robot">
+<robot xmlns:xacro="http://www.ros.org/wiki/xacro" name="growbot">
 <xacro:macro name="arm" params="prefix radius length reflect">
     <!-- rpy (roll pitch yaw) describes rotation in radians -->
     <!-- xyz describes translation in meters -->
-    <link name="${prefix}_arm">
+    <link name="${prefix}_wheel">
         <visual>
             <origin rpy="0 0 0" xyz="0 0 1"/> <!-- set the origin to 0 to recenter the link to the child_frame -->
@@ -23,17 +23,17 @@
         </inertial>
     </link>
-    <joint name="base_to_${prefix}_arm" type="continuous">
+    <joint name="base_to_${prefix}_wheel" type="continuous">
         <axis xyz="0 1 0"/>
         <parent link="base_link"/>
-        <child link="${prefix}_arm"/>
+        <child link="${prefix}_wheel"/>
         <origin rpy="0.2 0 0" xyz="0 ${reflect*0.7} 0"/> <!-- move the child_frame with respect to parent_frame -->
         <limit effort="30" velocity="1.0"/>
     </joint>
-    <transmission name="${prefix}_arm_transmission">
+    <transmission name="${prefix}_wheel_transmission">
         <type>transmission_interface/SimpleTransmission</type>
         <actuator name="$${prefix}_motor">
             <mechanicalReduction>1</mechanicalReduction>
         </actuator>
-        <joint name="base_to_${prefix}_arm">
+        <joint name="base_to_${prefix}_wheel">
             <hardwareInterface>hardware_interface/VelocityJointInterface</hardwareInterface>
         </joint>
